File: SICKWATCH1/_autosave-UC.sch (KiCad schematic (older format))
At the start: 31 parts, among them SW1 SW_Push, U1 STM32F103C8Tx, Y1 Crystal

Commit message: Layout done (I GUESS)
Other:
- note added: "yd3414\n"
Changed lines of the file:
@@
 Text Notes 10400 4150 0    50   ~ 0
 UART Interface\n
+Text Notes 8350 3250 0    50   ~ 0
+yd3414\n
 $EndSCHEMATC
