File: SICKWATCH1/LED.sch (KiCad schematic (older format))
At the start: 22 parts, among them Q2 BSS138, Q3 BSS138

Commit message: fixed screenprints
Changed lines of the file:
@@
 Wire Wire Line
 	4950 6450 5100 6450
-Text HLabel 4100 5750 0    50   Input ~ 0
-K0
-Text HLabel 4100 6150 0    50   Input ~ 0
-K1
 Wire Wire Line
 	4400 6150 4800 6150
@@
 Text GLabel 1600 2200 0    50   Input ~ 0
 3V3
+Text GLabel 4100 5750 0    50   Input ~ 0
+K0
+Text GLabel 4100 6150 0    50   Input ~ 0
+K1
 $EndSCHEMATC

Commit message: finished V1.0 and ordered pcbs
Parts:
- C10: value C -> 100n
Changed lines of the file:
@@
 P 1950 2350
 F 0 "C10" H 2065 2396 50  0000 L CNN
-F 1 "C" H 2065 2305 50  0000 L CNN
+F 1 "100n" H 2065 2305 50  0000 L CNN
 F 2 "Capacitor_SMD:C_0603_1608Metric" H 1988 2200 50  0001 C CNN
 F 3 "~" H 1950 2350 50  0001 C CNN
