File: SICKWATCH1/UC.sch (KiCad schematic (older format))
At the start: 31 parts, among them SW1 SW_Push, U1 STM32F103C8Tx, Y1 Crystal

Commit message: finished V1.0 and ordered pcbs
Parts:
- added C15: 100n, Capacitor_SMD:C_0603_1608Metric, symbol Device:C
- added TP11: BUZ, TestPoint:TestPoint_Pad_D1.0mm, symbol Connector:TestPoint
- C1, C2: value C -> 33p
- C6: value C -> 1u
- R8: value R -> 10k
- R9: value R -> 1k
- TP2: value SWDIO -> DIO
- TP3: value SWCLK -> CLK
Connections:
- net GNDD: now also C15.2
- net at R7.1, U1.7 (NRST): now also C15.1
- net BUZ: now reaches U1.25 (PB12)
- net BUZ: now also TP11.1
Other:
- note added: "yd3414\n"
- moved on the sheet: R7
Changed lines of the file:
@@
 P 4300 3000
 F 0 "C1" V 4048 3000 50  0000 C CNN
-F 1 "C" V 4139 3000 50  0000 C CNN
+F 1 "33p" V 4139 3000 50  0000 C CNN
 F 2 "Capacitor_SMD:C_0603_1608Metric" H 4338 2850 50  0001 C CNN
 F 3 "~" H 4300 3000 50  0001 C CNN
@@
 P 4300 3300
 F 0 "C2" V 4048 3300 50  0000 C CNN
-F 1 "C" V 4139 3300 50  0000 C CNN
+F 1 "33p" V 4139 3300 50  0000 C CNN
 F 2 "Capacitor_SMD:C_0603_1608Metric" H 4338 3150 50  0001 C CNN
 F 3 "~" H 4300 3300 50  0001 C CNN
@@
 P 8350 4650
 F 0 "TP2" V 8304 4838 50  0000 L CNN
-F 1 "SWDIO" V 8395 4838 50  0000 L CNN
+F 1 "DIO" V 8395 4838 50  0000 L CNN
 F 2 "TestPoint:TestPoint_Pad_D1.0mm" H 8550 4650 50  0001 C CNN
 F 3 "~" H 8550 4650 50  0001 C CNN
@@
 P 8350 4950
 F 0 "TP3" V 8304 5138 50  0000 L CNN
-F 1 "SWCLK" V 8395 5138 50  0000 L CNN
+F 1 "CLK" V 8395 5138 50  0000 L CNN
 F 2 "TestPoint:TestPoint_Pad_D1.0mm" H 8550 4950 50  0001 C CNN
 F 3 "~" H 8550 4950 50  0001 C CNN
@@
 P 7700 3550
 F 0 "C6" H 7815 3596 50  0000 L CNN
-F 1 "C" H 7815 3505 50  0000 L CNN
+F 1 "1u" H 7815 3505 50  0000 L CNN
 F 2 "Capacitor_SMD:C_0603_1608Metric" H 7738 3400 50  0001 C CNN
 F 3 "~" H 7700 3550 50  0001 C CNN
@@
 P 7700 2850
 F 0 "R9" H 7770 2896 50  0000 L CNN
-F 1 "R" H 7770 2805 50  0000 L CNN
+F 1 "1k" H 7770 2805 50  0000 L CNN
 F 2 "Resistor_SMD:R_0603_1608Metric" V 7630 2850 50  0001 C CNN
 F 3 "~" H 7700 2850 50  0001 C CNN
@@
 L Device:R R7
 U 1 1 5CDAADD2
-P 5150 2050
-F 0 "R7" H 5220 2096 50  0000 L CNN
-F 1 "R" H 5220 2005 50  0000 L CNN
-F 2 "Resistor_SMD:R_0603_1608Metric" V 5080 2050 50  0001 C CNN
-F 3 "~" H 5150 2050 50  0001 C CNN
-	1    5150 2050
+P 4850 1050
+F 0 "R7" H 4920 1096 50  0000 L CNN
+F 1 "R" H 4920 1005 50  0000 L CNN
+F 2 "Resistor_SMD:R_0603_1608Metric" V 4780 1050 50  0001 C CNN
+F 3 "~" H 4850 1050 50  0001 C CNN
+	1    4850 1050
 	1    0    0    -1
 $EndComp
@@
 L power:GNDD #PWR04
 U 1 1 5CDABAEB
-P 5150 2200
-F 0 "#PWR04" H 5150 1950 50  0001 C CNN
-F 1 "GNDD" H 5154 2045 50  0000 C CNN
-F 2 "" H 5150 2200 50  0001 C CNN
-F 3 "" H 5150 2200 50  0001 C CNN
-	1    5150 2200
-	1    0    0    -1
-$EndComp
-Wire Wire Line
-	5350 1900 5150 1900
-Wire Wire Line
-	5350 1900 5350 2300
+P 4850 1300
+F 0 "#PWR04" H 4850 1050 50  0001 C CNN
+F 1 "GNDD" H 4854 1145 50  0000 C CNN
+F 2 "" H 4850 1300 50  0001 C CNN
+F 3 "" H 4850 1300 50  0001 C CNN
+	1    4850 1300
+	1    0    0    -1
+$EndComp
 $Comp
 L Device:R R3
@@
 P 7450 3550
 F 0 "R8" H 7520 3596 50  0000 L CNN
-F 1 "R" H 7520 3505 50  0000 L CNN
+F 1 "10k" H 7520 3505 50  0000 L CNN
 F 2 "Resistor_SMD:R_0603_1608Metric" V 7380 3550 50  0001 C CNN
 F 3 "~" H 7450 3550 50  0001 C CNN
@@
 Text Notes 10400 4150 0    50   ~ 0
 UART Interface\n
+Text Notes 8350 3250 0    50   ~ 0
+yd3414\n
+$Comp
+L Device:C C15
+U 1 1 5DDEAFBA
+P 5100 1050
+F 0 "C15" H 5215 1096 50  0000 L CNN
+F 1 "100n" H 5215 1005 50  0000 L CNN
+F 2 "Capacitor_SMD:C_0603_1608Metric" H 5138 900 50  0001 C CNN
+F 3 "~" H 5100 1050 50  0001 C CNN
+	1    5100 1050
+	1    0    0    -1
+$EndComp
+Wire Wire Line
+	4850 1300 4850 1200
+Wire Wire Line
+	5100 1200 4850 1200
+Connection ~ 4850 1200
+Wire Wire Line
+	5350 900  5100 900
+Wire Wire Line
+	5350 900  5350 2300
+Connection ~ 5100 900
+Wire Wire Line
+	5100 900  4850 900
+Text Notes 9400 2800 0    50   ~ 0
+PROGRAMMING INTERFACE
+$Comp
+L Connector:TestPoint TP11
+U 1 1 5DE65D89
+P 9850 3000
+F 0 "TP11" V 9804 3187 50  0000 L CNN
+F 1 "BUZ" V 9895 3187 50  0000 L CNN
+F 2 "TestPoint:TestPoint_Pad_D1.0mm" H 10050 3000 50  0001 C CNN
+F 3 "~" H 10050 3000 50  0001 C CNN
+	1    9850 3000
+	0    1    1    0
+$EndComp
+Text GLabel 9850 3000 0    50   Input ~ 0
+BUZ
+Text GLabel 5350 4600 0    50   Input ~ 0
+BUZ
 $EndSCHEMATC
